File: PCB/PCB.kicad_pcb (KiCad board)
At the start: 4 copper layers, 21 x 51 mm, 33 parts, among them J1 USB_C_Receptacle_USB2.0_16P, J2 Conn_01x20, J3 Conn_01x20, SW1 SW_Push, U1 RP2040, U2 MCP1700x-330xxTT, U3 W25Q128JVS, Y1 Crystal_GND24

Commit message: Cleaning up production Data, and replacing flash memory to prepare for production. Ready for production.
Parts:
- U3: footprint Package_SON:Winbond_USON-8-1EP_3x2mm_P0.5mm_EP0.2x1.6mm -> lcsc_footprints:C7466821_USON8_L3_0-W2_0-P0_50-BL-EP
- moved C3 0.36 mm to (127.3, 63.3)
- moved C7 0.23 mm to (130.0, 57.9)
- turned U3 to -90 degrees
Connections:
- J3 pad 8: GND -> unconnected-(J3-Pin_8-Pad8)
Routing:
- net +3.3V: track 84.1 -> 84.9 mm

Commit message: finishing up project with BOM and FAB complete and clean.
Parts:
- J2, J3: footprint Connector_PinHeader_2.54mm:PinHeader_1x20_P2.54mm_Vertical -> lcsc_footprints:C50981_HDR-TH_20P-P2_54-V-M-1; moved to F.Cu
- moved J2 24.1 mm to (123.1, 62.7), turned to -90 degrees
- moved J3 24.1 mm to (140.8, 62.7), turned to -90 degrees
