File: PCB/PCB.kicad_sch (KiCad schematic)
At the start: 32 parts, among them J1 USB_C_Receptacle_USB2.0_16P, J2 Conn_01x20, J3 Conn_01x20, SW1 SW_Push, U1 RP2040, U2 MCP1700x-330xxTT, U3 W25Q128JVS, Y1 Crystal_GND24

Commit message: Almost Done with PCB
Parts:
- added R7: 1k, PCM_JLCPCB:R_0402, symbol Device:R_Small
- C1, C10, C11, C12, C13, C14, C15, C16, C17, C2, C3, C4, C5, C6, C7, C8, C9: footprint (none) -> Capacitor_SMD:C_0402_1005Metric
- J1: footprint (none) -> Connector_USB:USB_C_Receptacle_HCTL_HC-TYPE-C-16P-01A
- J2, J3: footprint (none) -> Connector_PinHeader_2.54mm:PinHeader_1x20_P2.54mm_Vertical
- R1, R2, R3, R4, R5, R6: footprint (none) -> PCM_JLCPCB:R_0402
- SW1: footprint (none) -> lcsc_footprints:C720477_SW-SMD_L3_9-W3_0-P4_45
- U3: footprint Package_SO:SOIC-8_5.3x5.3mm_P1.27mm -> Package_SON:Winbond_USON-8-1EP_3x2mm_P0.5mm_EP0.2x1.6mm
- Y1: footprint (none) -> lcsc_footprints:C9002_CRYSTAL-SMD_4P-L3_2-W2_5-BL
Connections:
- net QSPI_SCLK: now also U1.52 (QSPI_SCLK); no longer U1.53 (QSPI_SD0)
- net QSPI_SD0: now also U1.53 (QSPI_SD0); no longer U1.55 (QSPI_SD1)
- net QSPI_SD1: now also U1.55 (QSPI_SD1); no longer U1.54 (QSPI_SD2)
- net QSPI_SD2: now also U1.54 (QSPI_SD2); no longer U1.51 (QSPI_SD3)
- net QSPI_SD3: now also U1.51 (QSPI_SD3); no longer U1.52 (QSPI_SCLK)
- net SWCLK: now also H1.3; no longer H1.1
- net SWD: now also H1.1; no longer H1.3
- net XOUT: now also R7.2; no longer C15.1, Y1.1
- new net: C15.1, R7.1, Y1.1
Other:
- moved on the sheet: H1
Changed lines of the file:
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@@
 	)
 	(junction
-		(at 69.85 64.77)
+		(at 146.05 29.21)
 		(diameter 0)
 		(color 0 0 0 0)
 	)
 	(junction
-		(at 146.05 29.21)
+		(at 69.85 64.77)
 		(diameter 0)
 		(color 0 0 0 0)
@@
 	)
 	(junction
+		(at 105.41 101.6)
+		(diameter 0)
+		(color 0 0 0 0)
+	)
+	(junction
 		(at 156.21 24.13)
 		(diameter 0)
@@
 	)
 	(junction
-		(at 105.41 101.6)
-		(diameter 0)
-		(color 0 0 0 0)
-	)
-	(junction
 		(at 194.31 29.21)
 		(diameter 0)
@@
 	(wire
 		(pts
-			(xy 102.87 101.6) (xy 105.41 101.6)
+			(xy 96.52 101.6) (xy 97.79 101.6)
 		)
 		(stroke
@@
 	(wire
 		(pts
+			(xy 102.87 101.6) (xy 105.41 101.6)
+		)
+		(stroke
+			(width 0)
+			(type default)
+		)
+	)
+	(wire
+		(pts
 			(xy 153.67 46.99) (xy 156.21 46.99)
 		)
@@
 	)
 	(label "XOUT"
-		(at 102.87 101.6 180)
+		(at 96.52 101.6 180)
 		(effects
 			(font
@@
 		)
 	)
-	(label "QSPI_SCLK"
-		(at 142.24 69.85 180)
-		(effects
-			(font
-				(size 1.27 1.27)
-			)
-			(justify right bottom)
-		)
-	)
 	(label "XIN"
 		(at 142.24 100.33 180)
@@
 		)
 	)
+	(label "QSPI_SCLK"
+		(at 142.24 81.28 180)
+		(effects
+			(font
+				(size 1.27 1.27)
+			)
+			(justify right bottom)
+		)
+	)
 	(label "XOUT"
 		(at 142.24 105.41 180)
@@
 	)
 	(label "QSPI_SD3"
-		(at 142.24 81.28 180)
+		(at 142.24 77.47 180)
 		(effects
 			(font
@@
 	)
 	(label "QSPI_SD1"
-		(at 142.24 74.93 180)
+		(at 142.24 72.39 180)
 		(effects
 			(font
@@
 	)
 	(label "QSPI_SD2"
-		(at 142.24 77.47 180)
+		(at 142.24 74.93 180)
 		(effects
 			(font
@@
 	)
 	(label "QSPI_SD0"
-		(at 142.24 72.39 180)
+		(at 142.24 69.85 180)
 		(effects
 			(font
@@
 			)
 		)
-		(property "Footprint" ""
+		(property "Footprint" "Capacitor_SMD:C_0402_1005Metric"
 			(at 146.05 26.67 0)
 			(hide yes)
@@
 			)
 		)
-		(property "Footprint" ""
+		(property "Footprint" "lcsc_footprints:C9002_CRYSTAL-SMD_4P-L3_2-W2_5-BL"
 			(at 115.57 101.6 0)
 			(hide yes)
@@
 			)
 		)
-		(property "Footprint" ""
+		(property "Footprint" "Connector_PinHeader_2.54mm:PinHeader_1x20_P2.54mm_Vertical"
 			(at 77.47 128.27 0)
 			(hide yes)
@@
 			)
 		)
-		(property "Footprint" ""
+		(property "Footprint" "Capacitor_SMD:C_0402_1005Metric"
 			(at 102.87 44.45 0)
 			(hide yes)
@@
 			)
 		)
-		(property "Footprint" ""
+		(property "Footprint" "Capacitor_SMD:C_0402_1005Metric"
 			(at 204.47 26.67 0)
 			(hide yes)
@@
 			)
 		)
-		(property "Footprint" ""
+		(property "Footprint" "PCM_JLCPCB:R_0402"
 			(at 74.93 52.07 0)
 			(hide yes)
@@
 			)
 		)
-		(property "Footprint" ""
+		(property "Footprint" "PCM_JLCPCB:R_0402"
 			(at 212.09 54.61 0)
 			(hide yes)
@@
 			)
 		)
-		(property "Footprint" ""
+		(property "Footprint" "PCM_JLCPCB:R_0402"
 			(at 66.04 52.07 0)
 			(hide yes)
@@
 			)
 		)
-		(property "Footprint" "Package_SO:SOIC-8_5.3x5.3mm_P1.27mm"
+		(property "Footprint" "Package_SON:Winbond_USON-8-1EP_3x2mm_P0.5mm_EP0.2x1.6mm"
 			(at 96.52 49.53 0)
 			(hide yes)
@@
 			)
 		)
-		(property "Footprint" ""
+		(property "Footprint" "Capacitor_SMD:C_0402_1005Metric"
 			(at 135.89 26.67 0)
 			(hide yes)
@@
 			)
 		)
-		(property "Footprint" ""
+		(property "Footprint" "lcsc_footprints:C720477_SW-SMD_L3_9-W3_0-P4_45"
 			(at 62.23 72.39 0)
 			(hide yes)
@@
 			)
 		)
-		(property "Footprint" ""
+		(property "Footprint" "Capacitor_SMD:C_0402_1005Metric"
 			(at 101.6 59.69 0)
 			(hide yes)
@@
 			)
 		)
-		(property "Footprint" ""
+		(property "Footprint" "Capacitor_SMD:C_0402_1005Metric"
 			(at 184.15 26.67 0)
 			(hide yes)
@@
 			)
 		)
-		(property "Footprint" ""
+		(property "Footprint" "Capacitor_SMD:C_0402_1005Metric"
 			(at 105.41 104.14 0)
 			(hide yes)
@@
 			)
 		)
-		(property "Footprint" ""
+		(property "Footprint" "Capacitor_SMD:C_0402_1005Metric"
 			(at 214.63 26.67 0)
 			(hide yes)
@@
 			)
 		)
-		(property "Footprint" ""
+		(property "Footprint" "PCM_JLCPCB:R_0402"
 			(at 69.85 62.23 0)
 			(hide yes)
@@
 			)
 		)
-		(property "Footprint" ""
+		(property "Footprint" "Capacitor_SMD:C_0402_1005Metric"
 			(at 128.27 26.67 0)
 			(hide yes)
@@
 			)
 		)
-		(property "Footprint" ""
+		(property "Footprint" "Capacitor_SMD:C_0402_1005Metric"
 			(at 234.95 26.67 0)
 			(hide yes)
@@
 			)
 		)
-		(property "Footprint" ""
+		(property "Footprint" "Connector_PinHeader_2.54mm:PinHeader_1x20_P2.54mm_Vertical"
 			(at 41.91 128.27 0)
 			(hide yes)
@@
 			)
 		)
-		(property "Footprint" ""
+		(property "Footprint" "Capacitor_SMD:C_0402_1005Metric"
 			(at 224.79 26.67 0)
 			(hide yes)
@@
 			)
 		)
-		(property "Footprint" ""
+		(property "Footprint" "Capacitor_SMD:C_0402_1005Metric"
 			(at 194.31 26.67 0)
 			(hide yes)
@@
 			)
 		)
-		(property "Footprint" ""
+		(property "Footprint" "Capacitor_SMD:C_0402_1005Metric"
 			(at 163.83 26.67 0)
 			(hide yes)
@@
 			)
 		)
-		(property "Footprint" ""
+		(property "Footprint" "Connector_USB:USB_C_Receptacle_HCTL_HC-TYPE-C-16P-01A"
 			(at 41.91 57.15 0)
 			(hide yes)
@@
 			)
 		)
-		(property "Footprint" ""
+		(property "Footprint" "PCM_JLCPCB:R_0402"
 			(at 227.33 57.15 0)
 			(hide yes)
@@
 	)
 	(symbol
+		(lib_id "Device:R_Small")
+		(at 100.33 101.6 270)
+		(unit 1)
+		(body_style 1)
+		(exclude_from_sim no)
+		(in_bom yes)
+		(on_board yes)
+		(in_pos_files yes)
+		(dnp no)
+		(fields_autoplaced yes)
+		(property "Reference" "R7"
+			(at 100.33 96.52 90)
+			(show_name no)
+			(do_not_autoplace no)
+			(effects
+				(font
+					(size 1.016 1.016)
+				)
+			)
+		)
+		(property "Value" "1k"
+			(at 100.33 99.06 90)
+			(show_name no)
+			(do_not_autoplace no)
+			(effects
+				(font
+					(size 1.27 1.27)
+				)
+			)
+		)
+		(property "Footprint" "PCM_JLCPCB:R_0402"
+			(at 100.33 101.6 0)
+			(hide yes)
+			(show_name no)
+			(do_not_autoplace no)
+			(effects
+				(font
+					(size 1.27 1.27)
+				)
+			)
+		)
+		(property "Datasheet" ""
+			(at 100.33 101.6 0)
+			(hide yes)
+			(show_name no)
+			(do_not_autoplace no)
+			(effects
+				(font
+					(size 1.27 1.27)
+				)
+			)
+		)
+		(property "Description" "Resistor, small symbol"
+			(at 100.33 101.6 0)
+			(hide yes)
+			(show_name no)
+			(do_not_autoplace no)
+			(effects
+				(font
+					(size 1.27 1.27)
+				)
+			)
+		)
+		(pin "2"
+		)
+		(pin "1"
+		)
+		(instances
+			(project "PCB"
+				(path "/0ca16757-d282-4856-b58b-7fb83f3c2bb4"
+					(reference "R7")
+					(unit 1)
+				)
+			)
+		)
+	)
+	(symbol
 		(lib_id "Device:C_Small")
 		(at 80.01 44.45 0)
@@
 			)
 		)
-		(property "Footprint" ""
+		(property "Footprint" "Capacitor_SMD:C_0402_1005Metric"
 			(at 80.01 44.45 0)
 			(hide yes)
@@
 			)
 		)
-		(property "Footprint" ""
+		(property "Footprint" "Capacitor_SMD:C_0402_1005Metric"
 			(at 156.21 26.67 0)
 			(hide yes)
@@
 			)
 		)
-		(property "Footprint" ""
+		(property "Footprint" "PCM_JLCPCB:R_0402"
 			(at 67.31 74.93 0)
 			(hide yes)
@@
 			)
 		)
-		(property "Footprint" ""
+		(property "Footprint" "Capacitor_SMD:C_0402_1005Metric"
 			(at 173.99 26.67 0)
 			(hide yes)
@@
 	(symbol
 		(lib_id "FCFILES:PZ254V-11-03P_C2937625")
-		(at 58.42 149.86 90)
+		(at 58.42 149.86 270)
+		(mirror x)
 		(unit 1)
 		(body_style 1)
@@
 		(in_pos_files yes)
 		(dnp no)
-		(fields_autoplaced yes)
 		(property "Reference" "H1"
-			(at 64.77 148.5899 90)
+			(at 52.07 148.5899 90)
 			(show_name no)
 			(do_not_autoplace no)
@@
 		)
 		(property "Value" "Debug"
-			(at 64.77 151.1299 90)
+			(at 52.07 151.1299 90)
 			(show_name no)
 			(do_not_autoplace no)
@@
 		)
 		(property "Footprint" "lcsc_footprints:C2937625_HDR-TH_3P-P2_54-V-M_PZ254V-11-03P"
-			(at 68.58 149.86 0)
+			(at 48.26 149.86 0)
 			(hide yes)
 			(show_name no)
@@
 		)
 		(property "Datasheet" "https://wmsc.lcsc.com/wmsc/upload/file/pdf/v2/lcsc/2201121800_XFCN-PZ254V-11-03P_C2937625.pdf"
-			(at 58.293 152.146 0)
+			(at 58.547 152.146 0)
 			(hide yes)
 			(show_name no)
@@
 			)
 		)
-		(property "Footprint" ""
+		(property "Footprint" "Capacitor_SMD:C_0402_1005Metric"
 			(at 123.19 104.14 0)
 			(hide yes)

Commit message: Cleaning up production Data, and replacing flash memory to prepare for production. Ready for production.
Parts:
- U3: footprint Package_SON:Winbond_USON-8-1EP_3x2mm_P0.5mm_EP0.2x1.6mm -> lcsc_footprints:C7466821_USON8_L3_0-W2_0-P0_50-BL-EP
Changed lines of the file:
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@@
 			)
 		)
-		(property "Footprint" "Package_SON:Winbond_USON-8-1EP_3x2mm_P0.5mm_EP0.2x1.6mm"
+		(property "Footprint" "lcsc_footprints:C7466821_USON8_L3_0-W2_0-P0_50-BL-EP"
 			(at 96.52 49.53 0)
 			(hide yes)

Commit message: finishing up project with BOM and FAB complete and clean.
Parts:
- J2, J3: footprint Connector_PinHeader_2.54mm:PinHeader_1x20_P2.54mm_Vertical -> lcsc_footprints:C50981_HDR-TH_20P-P2_54-V-M-1
Changed lines of the file:
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@@
 			)
 		)
-		(property "Footprint" "Connector_PinHeader_2.54mm:PinHeader_1x20_P2.54mm_Vertical"
+		(property "Footprint" "lcsc_footprints:C50981_HDR-TH_20P-P2_54-V-M-1"
 			(at 77.47 128.27 0)
 			(hide yes)
@@
 			)
 		)
-		(property "Footprint" "Connector_PinHeader_2.54mm:PinHeader_1x20_P2.54mm_Vertical"
+		(property "Footprint" "lcsc_footprints:C50981_HDR-TH_20P-P2_54-V-M-1"
 			(at 41.91 128.27 0)
 			(hide yes)
